File: Hardware/proton.sch (EAGLE design)
At the start: 101 parts, among them IC1 MCP2300X/SO, IC2 MAX7219CWG, IC3 LD117AS33TR, J1 POWER_JACKPTH_LOCK, K1 ZF112, M2 WIRELESS-NRF24L01, P1 P120PK, Q1 BSS138, Q2 BSS138, SW1 ENCODER_SW1-PEC12, T1 BC847, T2 BC847, T3 BC847, U1 LCD-16X2SILK, U2 I2C EEPROM

Commit message: Power rails and toggle switch
Parts:
- added J2, J3: (no value), SparkFun-Connectors:CONN_05JST-VERT
- added J4, J5: (no value), SparkFun-Connectors:CONN_10X2NOSILK
- added S10: (no value), switch:M9040P
- SW1: value ENCODER_SW1-PEC12 -> ENCODER
Connections:
- removed net 5V: U$10.VCC, U$9.VCC
- removed net N$2: J1.PWR, U$11.IN+
- new net +12V: J1.PWR, J5.10, J5.12, J5.14, J5.16, J5.18, J5.2, J5.20, J5.4, J5.6, J5.8, S10.P
- new net N$82: J3.5, ULN1.16
- new net N$83: J3.4, ULN1.15
- new net N$84: J3.3, ULN1.14
- new net N$85: J3.2, ULN1.13
- new net N$86: J3.1, ULN1.12
- new net N$87: J2.1, ULN1.7
- new net N$88: J2.2, ULN1.6
- new net N$89: J2.3, ULN1.5
- new net N$90: J2.4, ULN1.4
- new net N$91: J2.5, ULN1.3
- net +5V: now also J5.1, J5.11, J5.13, J5.15, J5.17, J5.19, J5.3, J5.5, J5.7, J5.9, U$10.VCC, U$9.VCC
- net 3.3V: now also J4.10, J4.12, J4.14, J4.16, J4.18, J4.2, J4.20, J4.4, J4.6, J4.8
- net GND: now also J1.GND, J1.GNDBREAK, J4.1, J4.11, J4.13, J4.15, J4.17, J4.19, J4.3, J4.5, J4.7, J4.9, U$11.IN-
- net N$3: now also S10.S, U$11.IN+; no longer J1.GND, J1.GNDBREAK, U$11.IN-

Commit message: properly sorted the pin-distributions, changed the motor drievr
Parts:
- removed J4, J5: (no value), SparkFun-Connectors:CONN_10X2NOSILK
- removed S6, S8, S9: DTSM-6, switch-tact:DTSM-6
- removed SG1: BMT1205XH7.5, buzzer:BMT1205XH7.5
- removed ULN1: (no value), SparkFun-IC-Special-Function:ULN2803DIP
- added BUZZER: BMT1205XH7.5, buzzer:BMT1205XH7.5
- added C16: 100nf, SparkFun:CAP0805
- added C17, C18, C19, C20: .1ufF, SparkFun:CAP0805
- added IC4: L293D, st-microelectronics:L293D
- added S11: (no value), switch-dil:DIP10YL
- added S12: (no value), switch-dil:DIP08YL
- added S14: (no value), switch-dil:DIP06YL
- J2, J3: device SparkFun-Connectors:CONN_05JST-VERT -> SparkFun-Connectors:CONN_05X2NO_SILK
- LED1: value Blue -> Yellow
- S1: value (none) -> DTSM-6; device switch-dil:DIP10YL -> switch-tact:DTSM-6
- S2: value (none) -> DTSM-6; device switch-dil:DIP08YL -> switch-tact:DTSM-6
- S3: value (none) -> DTSM-6; device switch-dil:DIP03YL -> switch-tact:DTSM-6; OC_FARNELL unknown -> (none); OC_NEWARK unknown -> (none)
- S4: device switch-dil:DIP06YL -> switch-dil:DIP05YL
- renumbered LED8 to LED1, U$7 to T/H
Connections:
- removed net N$82: J3.5, ULN1.16
- removed net N$83: J3.4, ULN1.15
- removed net N$84: J3.3, ULN1.14
- removed net N$85: J3.2, ULN1.13
- removed net N$86: J3.1, ULN1.12
- removed net N$87: J2.1, ULN1.7
- removed net N$88: J2.2, ULN1.6
- removed net N$89: J2.3, ULN1.5
- removed net N$90: J2.4, ULN1.4
- removed net N$91: J2.5, ULN1.3
- new net A6: P1G$1.S, S4.7
- new net A7: R12.P$1, R13.1, S4.6
- new net N$9: C18.2, IC4.3Y, U$13.CON2
- net +12V: now also J3.10, J3.2, J3.4, J3.6, J3.8; no longer J5.10, J5.12, J5.14, J5.16, J5.18, J5.2, J5.20, J5.4, J5.6, J5.8
- net +5V: now also BUZZER.+, C16.1, IC4.1-2EN, IC4.3-4EN, IC4.VCC1, IC4.VCC2, J3.1, J3.3, J3.5, J3.7, J3.9; no longer J5.1, J5.11, J5.13, J5.15, J5.17, J5.19, J5.3, J5.5, J5.7, J5.9, SG1.+, ULN1.10
- net -A0: now also S14.6; no longer S4.6
- net -A1: now also S14.5; no longer S4.5
- net -A2: now also S14.4; no longer S4.4
- net -A3: now also S14.3; no longer S4.3
- net -A6: now also S4.4
- net -A7: now also S4.5
- net -AREF: now also S11.3; no longer S1.3
- net -D10: now also S11.8; no longer S1.8
- net -D11: now also M2.MOSI, S11.7, S5.1; no longer S1.7
- net -D12: now also M2.MISO, S11.6, S5.3; no longer S1.6
- net -D13: now also M2.SCK, S11.5, S5.2; no longer S1.5
- net -D2: now also S12.6; no longer S2.6
- net -D3: now also S12.5; no longer S2.5
- net -D4: now also S12.4; no longer S2.4
- net -D5: now also S12.3; no longer S2.3
- net -D6: now also S12.2; no longer S2.2
- net -D7: now also S12.1; no longer S2.1
- net -D8: now also S11.10; no longer S1.10
- net -D9: now also S11.9; no longer S1.9
- net -RX: now also S12.8; no longer S2.8
- net -SCL: now also S11.1, S14.1; no longer S1.1, S4.1
- net -SDA: now also S11.2, S14.2; no longer S1.2, S4.2
- net -TX: now also S12.7; no longer S2.7
- net 3.3V: now also J2.10, J2.2, J2.4, J2.6, J2.8; no longer J4.10, J4.12, J4.14, J4.16, J4.18, J4.2, J4.20, J4.4, J4.6, J4.8
- net A0: now also IC4.1A, S14.7; no longer P1G$1.S, S4.7
- net A1: now also R31.1, S14.8, S2.1, S2.2, S3.1, S3.2, SW1SW.1; no longer R24.1, S4.8
- net A2: now also R26.1, S14.9, T/H.DATA; no longer R12.P$1, R13.1, S4.9
- net A3: now also S14.10; no longer S4.10
- net A4: now also S14.11; no longer S4.11
- net A5: now also S14.12; no longer R31.1, S4.12, S8.1, S8.2, S9.1, S9.2, SW1SW.1
- net AREF: now also S11.18; no longer S1.18
- net D10: now also S11.13, S4.3; no longer S1.13, S3.3
- net D11: now also S11.14, S4.2; no longer S1.14, S3.2, S5.1
- net D12: now also S11.15, S4.1; no longer S1.15, S3.1, S5.3
- net D13: now also S11.16; no longer S1.16, S5.2, ULN1.2
- net D2: now also R24.1, S12.11; no longer S2.11
- net D3: now also S12.12; no longer S2.12
- net D4: now also S12.13; no longer S2.13
- net D5: now also IC4.4A, S12.14; no longer S2.14, ULN1.1
- net D6: now also S12.15; no longer S2.15
- net D7: now also S12.16; no longer S2.16
- net D8: now also S1.1, S1.2, S11.11; no longer S1.11, S6.1, S6.2
- net D9: now also S11.12; no longer S1.12
- net GND: now also C16.2, C17.1, C18.1, C19.1, C20.1, IC4.2A, IC4.3A, IC4.GND1, IC4.GND2, IC4.GND3, IC4.GND4, J2.1, J2.3, J2.5, J2.7, J2.9, S1.3, S11.17, S11.4; no longer J4.1, J4.11, J4.13, J4.15, J4.17, J4.19, J4.3, J4.5, J4.7, J4.9, S1.17, S6.3, S6.4, U$12.CON2, U$13.CON2, ULN1.9
- net MISO: no longer M2.MISO
- net MOSI: no longer M2.MOSI
- net MOTOR1: now also C17.2, IC4.4Y; no longer ULN1.18
- net MOTOR2: now also C20.2, IC4.1Y; no longer ULN1.17
- net N$1: now also C19.2, IC4.2Y, U$12.CON2; no longer R26.1, T/H.DATA
- net N$11: now also S3.3, S3.4; no longer S9.3, S9.4
- net N$18: now also BUZZER.-; no longer SG1.-
- net N$5: now also S2.3, S2.4; no longer S8.3, S8.4
- net RX: now also S12.9; no longer S2.9
- net SCK: no longer M2.SCK
- net SCL: now also S11.20; no longer S1.20
- net SDA: now also S11.19; no longer S1.19
- net S_D10: now also S4.8; no longer S3.4
- net S_D11: now also S4.9; no longer S3.5
- net S_D12: now also S4.10; no longer S3.6
- net TX: now also S12.10; no longer S2.10

Commit message: Fine tunings. Major change motor driver
Parts:
- added R30, R34: 1k, SparkFun:RESISTOR0805-RES
- renumbered JP2 to ESP, K1 to RELAY, M2 to NRF, P1 to POTENTIOMETER, R12 to PHOTOCELL, SW1 to SW4, T/H to TEMPERATURESENSOR, TSOP1 to IR, U$10 to ULTRASONIC, U$12 to MOTOR2, U$13 to MOTOR1, U$3 to XBEE, U$9 to PIR, U2 to EEPROM
Connections:
- net +5V: now also R30.1, R34.1
- net D6: now also R34.2
- net D7: now also R30.2
